File: DacBoard/DacBoard.kicad_pcb (KiCad board)
At the start: 0 parts

Commit message: Schematic finalized (for now); Begin PCB
Parts:
- added C1: 100n, Capacitor_SMD:C_0805_2012Metric_Pad1.18x1.45mm_HandSolder, F.Cu at (85.5, 64.0)
- added C10: 100n, Capacitor_SMD:C_0805_2012Metric_Pad1.18x1.45mm_HandSolder, F.Cu at (138.0, 72.0)
- added C11: 100n, Capacitor_SMD:C_0805_2012Metric_Pad1.18x1.45mm_HandSolder, F.Cu at (123.0, 72.0)
- added C2: 100n, Capacitor_SMD:C_0805_2012Metric_Pad1.18x1.45mm_HandSolder, F.Cu at (71.1, 69.5)
- added C3: 1u, Capacitor_SMD:C_0805_2012Metric_Pad1.18x1.45mm_HandSolder, F.Cu at (58.2, 71.1)
- added C4: 220n, Capacitor_SMD:C_0805_2012Metric_Pad1.18x1.45mm_HandSolder, F.Cu at (63.0, 71.1)
- added C5: 220n, Capacitor_SMD:C_0805_2012Metric_Pad1.18x1.45mm_HandSolder, F.Cu at (80.7, 67.0)
- added C6: 100n, Capacitor_SMD:C_0805_2012Metric_Pad1.18x1.45mm_HandSolder, F.Cu at (117.5, 72.0)
- added C7: 100n, Capacitor_SMD:C_0805_2012Metric_Pad1.18x1.45mm_HandSolder, F.Cu at (117.5, 87.5)
- added C8: 100n, Capacitor_SMD:C_0805_2012Metric_Pad1.18x1.45mm_HandSolder, F.Cu at (138.0, 86.0)
- added C9: 100n, Capacitor_SMD:C_0805_2012Metric_Pad1.18x1.45mm_HandSolder, F.Cu at (123.0, 86.0)
- added J1: DacConnector, Connector_PCBEdge:BUS_PCIexpress_x4, F.Cu at (101.0, 105.2)
- added R1: 6R2, Resistor_SMD:R_0805_2012Metric_Pad1.20x1.40mm_HandSolder, F.Cu at (67.8, 72.4)
- added R2: 6R2, Resistor_SMD:R_0805_2012Metric_Pad1.20x1.40mm_HandSolder, F.Cu at (80.7, 70.0)
- added RV1: 100k, Potentiometer_SMD:Potentiometer_Bourns_TC33X_Vertical, F.Cu at (95.3, 59.9)
- added RV2: 100k, Potentiometer_SMD:Potentiometer_Bourns_TC33X_Vertical, F.Cu at (80.3, 60.1)
- added U1: 74HC00, Package_SO:SOIC-14_3.9x8.7mm_P1.27mm, F.Cu at (111.0, 74.5)
- added U2: AD688, Package_SO:SOIC-16W_7.5x10.3mm_P1.27mm, F.Cu at (76.5, 81.0)
- added U3: 74HC00, Package_SO:SOIC-14_3.9x8.7mm_P1.27mm, F.Cu at (111.0, 90.0)
- added U4: AD5725, Package_SO:SSOP-28_5.3x10.2mm_P0.65mm, F.Cu at (130.5, 75.5)
- added U5: AD5725, Package_SO:SSOP-28_5.3x10.2mm_P0.65mm, F.Cu at (130.5, 89.5)
Routing:
- net GND: track 0.00 -> 52.4 mm
- net +15V: track 0.00 -> 9.67 mm
Other:
- board outline added: 34.3 x 8.4 mm
- copper layers 0 -> 2
