File: DacBoard/DacBoard.kicad_pcb (KiCad board)
At the start: 2 copper layers, 34.3 x 8.4 mm, 21 parts, among them J1 DacConnector, U1 74HC00, U2 AD688, U3 74HC00, U4 AD5725, U5 AD5725

Commit message: Working on PCB layout
Parts:
- moved C8 109.6 mm to (39.5, 38.0)
- moved C9 109.6 mm to (24.5, 38.0)
- moved RV1 107.9 mm to (-12.5, 55.0), turned to 90 degrees
- moved U4 104.7 mm to (32.0, 40.0)
- moved U5 104.4 mm to (32.0, 55.0)
- moved C10 100.3 mm to (39.5, 53.0)
- moved C11 100.3 mm to (24.5, 53.0)
- moved C1 95.7 mm to (-8.50, 46.0), turned to 90 degrees
- moved RV2 84.3 mm to (-4.00, 60.0)
- moved U2 82.2 mm to (0.00, 51.0)
- moved R1 78.0 mm to (-4.50, 43.0), turned to 180 degrees
- moved R2 74.4 mm to (9.00, 50.0), turned to 90 degrees
- moved C4 74.4 mm to (-8.50, 50.5), turned to -90 degrees
- moved C5 71.3 mm to (11.5, 50.0), turned to 90 degrees
- moved C3 68.6 mm to (-8.50, 55.0), turned to -90 degrees
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Connections:
- C6 pad 1: Net-(C6-Pad1) -> +5V
- C7 pad 1: Net-(C6-Pad1) -> +5V
- U3 pad 10: Net-(U3-Pad10) -> Net-(U3-Pad11)
- U3 pad 11: /~LDAC~_1 -> Net-(U3-Pad11)
- U3 pad 12: Net-(U3-Pad12) -> Net-(U3-Pad6)
- U3 pad 13: Net-(U3-Pad12) -> Net-(U3-Pad3)
- U3 pad 6: Net-(U3-Pad10) -> Net-(U3-Pad6)
- U3 pad 8: Net-(U3-Pad12) -> /~LDAC~_1
- U3 pad 9: Net-(U3-Pad3) -> Net-(U3-Pad11)
Routing:
- net GND: track 52.4 -> 19.7 mm
- net Net-(RV1-Pad3): track 0.00 -> 25.0 mm
- net /~LDAC: track 0.00 -> 22.5 mm, vias 0 -> 2
- net /A2: track 0.00 -> 18.7 mm, vias 0 -> 1
- net +5V: track 0.00 -> 17.3 mm
- net -15V: track 0.00 -> 13.6 mm
- net Net-(RV2-Pad2): track 0.00 -> 11.9 mm
- net Net-(RV1-Pad2): track 0.00 -> 8.64 mm
- net Net-(RV1-Pad1): track 0.00 -> 8.61 mm
- net Net-(U3-Pad6): track 0.00 -> 6.53 mm
- net Net-(U1-Pad10): track 0.00 -> 6.22 mm
- net Net-(U3-Pad3): track 0.00 -> 5.48 mm
- net Net-(R2-Pad2): track 0.00 -> 4.84 mm
- net /Vref+: track 0.00 -> 4.00 mm
- net Net-(C3-Pad1): track 0.00 -> 3.94 mm
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